File: 01 - FC_KiCadProj/ACwing_FC_H.kicad_pcb (KiCad board)
At the start: 4 copper layers, 40.8 x 40.8 mm, 108 parts, among them J1 USB-C (HRO TYPE-C-31-M-12), J2 ESC link, J3 Qwiic, J4 Qwiic, J5 ELRS, J6 ESC link B, J7 VBAT+, J8 GND, Q5 AO3401A, U1 LSM6DSV16X, U10 W25Q128JV, U11 LDK130PU-R, U12 LM5166DRCT, U2 STM32WB55CGU6, U3 IIS2MDC, U4 LPS22HB, U5 LD39130SPUR, U7 USBLC6-2SC6, U8 MLPF-WB55-01E3, Y1 32MHz

Commit message: Fix FC board rename
Parts:
- AE1: footprint DimaQuad:Johanson_2450AT18x100 -> ACwing:Johanson_2450AT18x100
- C1, C12, C14, C15, C16, C17, C18, C19, C21, C22, C23, C24, C25, C26, C27, C28, C29, C36, C39, C40, C41, C42, C43, C44, C45, C49, C8: footprint DimaQuad:C_0402_1005Metric -> ACwing:C_0402_1005Metric
- C2, C47, C6: footprint DimaQuad:C_1206_3216Metric -> ACwing:C_1206_3216Metric
- C20, C7, C9: footprint DimaQuad:C_0603_1608Metric -> ACwing:C_0603_1608Metric
- C46: footprint DimaQuad:C_0805_2012Metric -> ACwing:C_0805_2012Metric
- D1, D2, D3, D4: footprint DimaQuad:LED_WS2812B-2020_PLCC4_2.0x2.0mm -> ACwing:LED_WS2812B-2020_PLCC4_2.0x2.0mm
- D11: footprint DimaQuad:D_SOD-523 -> ACwing:D_SOD-523
- D9: footprint DimaQuad:D_SOD-123F -> ACwing:D_SOD-123F
- H1, H2, H3, H4: footprint DimaQuad:Grommet_PTH_3.2mm_Pad5.0mm -> ACwing:Grommet_PTH_3.2mm_Pad5.0mm
- J1: footprint DimaQuad:USB_C_Receptacle_HRO_TYPE-C-31-M-12 -> ACwing:USB_C_Receptacle_HRO_TYPE-C-31-M-12
- J2, J6: footprint DimaQuad:JST_SH_SM08B-SRSS-TB_1x08-1MP_P1.00mm_Horizontal -> ACwing:JST_SH_SM08B-SRSS-TB_1x08-1MP_P1.00mm_Horizontal
- J3, J4, J5: footprint DimaQuad:JST_SH_SM04B-SRSS-TB_1x04-1MP_P1.00mm_Horizontal -> ACwing:JST_SH_SM04B-SRSS-TB_1x04-1MP_P1.00mm_Horizontal
- J7, J8: footprint DimaQuad:TestPoint_Pad_2.0x2.0mm -> ACwing:TestPoint_Pad_2.0x2.0mm
- L1: footprint DimaQuad:L_0805_2012Metric -> ACwing:L_0805_2012Metric
- L2: footprint DimaQuad:L_0402_1005Metric -> ACwing:L_0402_1005Metric
- L3: footprint DimaQuad:L_Sunlord_SWPA5040S -> ACwing:L_Sunlord_SWPA5040S
- Q5: footprint DimaQuad:SOT-23 -> ACwing:SOT-23
- R10, R11, R12, R13, R14, R15, R16, R17, R18, R2, R20, R21, R22, R23, R24, R25, R26, R27, R28, R3, R34, R37, R38, R39, R4, R40, R41, R42, R47, R48, R8, R9: footprint DimaQuad:R_0402_1005Metric -> ACwing:R_0402_1005Metric
- TP1, TP2, TP3, TP4, TP5, TP6, TP7, TP8: footprint DimaQuad:TestPoint_Pad_D1.0mm -> ACwing:TestPoint_Pad_D1.0mm
- U1: footprint DimaQuad:LGA-14_3x2.5mm_P0.5mm_LayoutBorder3x4y -> ACwing:LGA-14_3x2.5mm_P0.5mm_LayoutBorder3x4y
- U10: footprint DimaQuad:WSON-8-1EP_6x5mm_P1.27mm_EP3.4x4mm -> ACwing:WSON-8-1EP_6x5mm_P1.27mm_EP3.4x4mm
- U11, U5: footprint DimaQuad:DFN-6_1.3x1.2mm_P0.4mm -> ACwing:DFN-6_1.3x1.2mm_P0.4mm
- U12: footprint DimaQuad:Texas_DRC0010J -> ACwing:Texas_DRC0010J
- U2: footprint DimaQuad:QFN-48-1EP_7x7mm_P0.5mm_EP5.6x5.6mm -> ACwing:QFN-48-1EP_7x7mm_P0.5mm_EP5.6x5.6mm
- U3: footprint DimaQuad:LGA-12_2x2mm_P0.5mm -> ACwing:LGA-12_2x2mm_P0.5mm
- U4: footprint DimaQuad:ST_HLGA-10_2x2mm_P0.5mm_LayoutBorder3x2y -> ACwing:ST_HLGA-10_2x2mm_P0.5mm_LayoutBorder3x2y
- U7: footprint DimaQuad:SOT-23-6 -> ACwing:SOT-23-6
- U8: footprint DimaQuad:ST_MLPF-WB55-01E3_CSP-6 -> ACwing:ST_MLPF-WB55-01E3_CSP-6
- Y1: footprint DimaQuad:Crystal_SMD_2016-4Pin_2.0x1.6mm -> ACwing:Crystal_SMD_2016-4Pin_2.0x1.6mm
