File: 01 - FC_KiCadProj/ACwing_FC_H.kicad_pcb (KiCad board)
At the start: 4 copper layers, 40.8 x 40.8 mm, 108 parts, among them J1 USB-C (HRO TYPE-C-31-M-12), J2 ESC link, J3 Qwiic, J4 Qwiic, J5 ELRS, J6 ESC link B, J7 VBAT+, J8 GND, Q5 AO3401A, U1 LSM6DSV16X, U10 W25Q128JV, U11 LDK130PU-R, U12 LM5166DRCT, U2 STM32WB55CGU6, U3 IIS2MDC, U4 LPS22HB, U5 LD39130SPUR, U7 USBLC6-2SC6, U8 MLPF-WB55-01E3, Y1 32MHz

Commit message: ACwing silkscreen: logos, board names, author, connector labels (DRC clean)
Co-Authored-By: Claude Opus 5.5 <noreply@anthropic.com>
Claude-Session: https://claude.ai/code/session_0189Xg6tRAL4bRZ656VQBtPX
Parts:
- added LOGO1: ACwing_Logo_Full_6mm, ACwing:ACwing_Logo_Full_6mm, F.Cu at (154.8, 96.5)
- added LOGO2: ACwing_Logo_Full_5mm, ACwing:ACwing_Logo_Full_5mm, B.Cu at (143.8, 83.3)
Other:
- board text added: "ACwing FC rev H"
- board text added: "Andrea Cirillo 2026"
- board text added: "BAT"
- board text added: "ELRS"
- board text added: "ESC A"
- board text added: "ESC B"
- board text added: "FC rev H"
- board text added: "FLOW"
- board text added: "GPS"
- board text added: "USB"

Commit message: Reorganize docs, regenerate outputs, remove author name from the PCBs
- fabrication outputs, schematics, STEP and PCB views moved to 00 - Docs/<board>_Docs
- single mechanical handoff and stack check in 04 - System_Docs, brand files in 05 - Brand
- silkscreen: ACwing logo, board name and labels only (no author name)

Co-Authored-By: Claude Opus 5.5 <noreply@anthropic.com>
Claude-Session: https://claude.ai/code/session_0189Xg6tRAL4bRZ656VQBtPX
Other:
- board text removed: "Andrea Cirillo 2026"
