File: 01 - FC_KiCadProj/ACwing_FC_A.kicad_sch (KiCad schematic)
At the start: 108 parts, among them J1 USB-C (HRO TYPE-C-31-M-12), J2 ESC link, J3 Qwiic, J4 Qwiic, J5 ELRS, J6 ESC link B, J7 VBAT+, J8 GND, Q5 AO3401A, U1 LSM6DSV16X, U10 W25Q128JV, U11 LDK130PU-R, U12 LM5166DRCT, U2 STM32WB55CGU6, U3 IIS2MDC, U4 LPS22HB, U5 LD39130SPUR, U7 USBLC6-2SC6, U8 MLPF-WB55-01E3, Y1 32MHz

Commit message: FC BoM fixes: R40 LCSC number, LPS22HH barometer, MCU sourcing note
- R40 47k 0402: C25819 (0603) -> C25792 (0402WGF4702TCE)
- U4: LPS22HBTR (out of stock) -> LPS22HHTR C2827824, same HLGA-10 footprint and pinout
- U2 STM32WB55CGU6 out of stock at LCSC/JLC: consigned part / Global Sourcing note

Co-Authored-By: Claude Opus 5.5 <noreply@anthropic.com>
Claude-Session: https://claude.ai/code/session_0189Xg6tRAL4bRZ656VQBtPX
Parts:
- U4: value LPS22HB -> LPS22HH; Note LPS22HBTR on the LPS22DF symbol/footprint (same HLGA-10 pin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 -> LPS22HHTR (replaces LPS22HBTR, same pinout) on the LPS22DF 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
Other:
- note added: "D - Sensors: LSM6DSV16X (SPI1) + sensor hub -> IIS2MDC, LPS22HH; log flash"
- note added: "Topology = IKS4A1 Mode 3: the IEKF firmware reads the IIS2MDC through the LSM6DSV16X sensor hub (samples aligned in the FIFO). Rev E: the IMU host interface is SPI; DRDY/INT2/baro INT not used (FIFO + timestamps) Addresses on the hub bus: IIS2MDC 0x1E, LPS22HH 0x5D"
- note removed: "D - Sensors: LSM6DSV16X (SPI1) + sensor hub -> IIS2MDC, LPS22HB; log flash"
- note removed: "Topology = IKS4A1 Mode 3: the IEKF firmware reads the IIS2MDC through the LSM6DSV16X sensor hub (samples aligned in the FIFO). Rev E: the IMU host interface is SPI; DRDY/INT2/baro INT not used (FIFO + timestamps) Addresses on the hub bus: IIS2MDC 0x1E, LPS22HB 0x5D"
Changed lines of the file:
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@@
       (type none))
 )
-  (text "D - Sensors: LSM6DSV16X (SPI1) + sensor hub -> IIS2MDC, LPS22HB; log flash"
+  (text "D - Sensors: LSM6DSV16X (SPI1) + sensor hub -> IIS2MDC, LPS22HH; log flash"
     (at 287.27 13.27 0)
     (effects
@@
           (size 1.27 1.27))
         (justify left)))
-    (property "Value" "LPS22HB"
+    (property "Value" "LPS22HH"
       (at 382.27 124.46 0)
       (effects
@@
         (font
           (size 1.27 1.27)) hide))
-    (property "Note" "LPS22HBTR on the LPS22DF symbol/footprint (same HLGA-10 pinout, pin 3 to GND). Optional. SA0 = 1 -> 0x5D"
+    (property "Note" "LPS22HHTR (replaces LPS22HBTR, same pinout) on the LPS22DF symbol/footprint (HLGA-10, pin 3 to GND). Optional. SA0 = 1 -> 0x5D"
       (at 377.19 109.22 0)
       (effects
@@
           (reference "#PWR087")
           (unit 1)))))
-  (text "Topology = IKS4A1 Mode 3: the IEKF firmware\nreads the IIS2MDC through the LSM6DSV16X\nsensor hub (samples aligned in the FIFO).\nRev E: the IMU host interface is SPI; DRDY/INT2/baro INT not used (FIFO + timestamps)\nAddresses on the hub bus: IIS2MDC 0x1E, LPS22HB 0x5D"
+  (text "Topology = IKS4A1 Mode 3: the IEKF firmware\nreads the IIS2MDC through the LSM6DSV16X\nsensor hub (samples aligned in the FIFO).\nRev E: the IMU host interface is SPI; DRDY/INT2/baro INT not used (FIFO + timestamps)\nAddresses on the hub bus: IIS2MDC 0x1E, LPS22HH 0x5D"
     (at 289.56 134.62 0)
     (effects

Commit message: FC: XL-2020RGBC-WS2812B LEDs, D11 Schottky replaced by 0R link R49
- D1-D4: XINGLIGHT XL-2020RGBC-WS2812B (C5349955), same footprint and pinout (WS2812B-2020 out of stock)
- D11 RB521S30 -> R49 0R 0402 at the same place: VLED = VSYS, LEDs above their 3.5 V minimum on 1S
- BoM, JLC BoM, CPL, schematic PDF, Gerber, STEP, PCB view regenerated; DRC 0

Co-Authored-By: Claude Opus 5.5 <noreply@anthropic.com>
Claude-Session: https://claude.ai/code/session_0189Xg6tRAL4bRZ656VQBtPX
Parts:
- D1, D2, D3, D4: value WS2812B-2020 -> XL-2020RGBC-WS2812B
- R49: renamed from D11; value RB521S30 -> 0R; footprint ACwing:D_SOD-523 -> ACwing:R_0402_1005Metric; symbol Device:D_Schottky -> Device:R; Note VLED = VSYS - 0.3 V: the LED data threshold (0.7 VLED) stay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 -> 0R link VSYS -> VLED (replaces the RB521S30 Schottky, 2026-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
Connections:
- net VLED: now also R49.2; no longer R49.1 (K)
- net VSYS: now also R49.1; no longer R49.2 (A)
Other:
- note added: "F - RGB LEDs (4 x XL-2020RGBC-WS2812B), programming pads, mounting"
- note removed: "F - RGB LEDs (4 x WS2812B), programming pads, mounting"
Changed lines of the file:
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@@
       (type none))
 )
-  (text "F - RGB LEDs (4 x WS2812B), programming pads, mounting"
+  (text "F - RGB LEDs (4 x XL-2020RGBC-WS2812B), programming pads, mounting"
     (at 287.27 155.27 0)
     (effects
@@
 )
   (symbol
-    (lib_id "Device:D_Schottky")
-    (at 358.14 162.56 180)
-    (unit 1)
-    (in_bom yes)
-    (on_board yes)
-    (dnp no)
-    (property "Reference" "D11"
+    (lib_id "Device:R")
+    (at 358.14 162.56 90)
+    (unit 1)
+    (in_bom yes)
+    (on_board yes)
+    (dnp no)
+    (property "Reference" "R49"
       (at 358.14 158.75 0)
       (effects
         (font
           (size 1.27 1.27))))
-    (property "Value" "RB521S30"
+    (property "Value" "0R"
       (at 358.14 166.37 0)
       (effects
         (font
           (size 1.27 1.27))))
-    (property "Footprint" "ACwing:D_SOD-523"
+    (property "Footprint" "ACwing:R_0402_1005Metric"
       (at 358.14 162.56 0)
       (effects
@@
         (font
           (size 1.27 1.27)) hide))
-    (property "Note" "VLED = VSYS - 0.3 V: the LED data threshold (0.7 VLED) stays below the 3.1 V GPIO level on USB too"
+    (property "Note" "0R link VSYS -> VLED (replaces the RB521S30 Schottky, 2026-10-27): VLED = VSYS keeps the XL-2020 LEDs above their 3.5 V minimum on 1S"
       (at 358.14 162.56 0)
       (effects
@@
       (project "ACwing_FC_A"
         (path "/7b987a65-9294-5c88-aa9e-83b05445a992"
-          (reference "D11")
+          (reference "R49")
           (unit 1)))))
   (symbol
@@
           (size 1.27 1.27))
         (justify left)))
-    (property "Value" "WS2812B-2020"
+    (property "Value" "XL-2020RGBC-WS2812B"
       (at 304.8 217.17 0)
       (effects
@@
           (size 1.27 1.27))
         (justify left)))
-    (property "Value" "WS2812B-2020"
+    (property "Value" "XL-2020RGBC-WS2812B"
       (at 327.66 217.17 0)
       (effects
@@
           (size 1.27 1.27))
         (justify left)))
-    (property "Value" "WS2812B-2020"
+    (property "Value" "XL-2020RGBC-WS2812B"
       (at 350.52 217.17 0)
       (effects
@@
           (size 1.27 1.27))
         (justify left)))
-    (property "Value" "WS2812B-2020"
+    (property "Value" "XL-2020RGBC-WS2812B"
       (at 373.38 217.17 0)
       (effects

Commit message: FC rev A: LED data level shifter U13, LEDs on VSYS (R49 removed)
- U13 SN74LV1T34DCKR (TI, LCSC C78541, SC-70-5) single-supply buffer powered
  from VSYS: TTL-level input (VIH <= 2.0 V), push-pull output at VSYS, so the
  XL-2020RGBC-WS2812B data input (VIH = 0.7 x VDD) is met on battery and on
  USB alone. C50 100 nF decoupling; R39 33R between U13 and D1.
- R49 0R removed: VLED merged into VSYS (LED supply unchanged in geometry,
  EMI at the magnetometer unchanged).
- PCB: U13/C50/R39 on the bottom next to D1, RGB data rerouted; DRC 0
  violations, 0 unconnected.
- BoM/JLC BoM/CPL (U13 correction 270 deg), costing, schematic PDF, Gerber,
  STEP, views regenerated; README and pin map updated.

Co-Authored-By: Claude Opus 5.5 <noreply@anthropic.com>
Claude-Session: https://claude.ai/code/session_0189Xg6tRAL4bRZ656VQBtPX
Parts:
- removed R49: 0R, ACwing:R_0402_1005Metric, symbol Device:R
- added C50: 100nF, ACwing:C_0402_1005Metric, symbol Device:C
- added U13: SN74LV1T34DCKR, ACwing:SOT-353_SC-70-5, symbol 74xGxx:74LVC1G34
- R39: Note Series resistor at the first LED input (data from PA7) -> Series resistor at the first LED input (data from U13)
Connections:
- net VLED is gone; now on net VSYS: C40.1, C41.1, C42.1, C45.1, D1.4 (VDD), D2.4 (VDD), D3.4 (VDD), D4.4 (VDD)
- net GND: now also C50.2, U13.3 (GND)
- net RGB_DIN: now also U13.2; no longer R39.1
- net VSYS: now also C50.1, U13.5 (VCC)
- new net RGB_DIN5: R39.1, U13.4
- no-connect marks 18 -> 19
