File: 02 - ESC_1S_KiCadProj/ACwing_ESC1S_B.kicad_pcb (KiCad board)
At the start: 4 copper layers, 40.8 x 40.8 mm, 49 parts, among them J1 ESC link, J2 BATT 1S, J4 USB-C (HRO TYPE-C-31-M-12), M1 coreless 8520, M2 coreless 8520, M3 coreless 8520, M4 coreless 8520, Q1 AON7524, Q2 AON7524, Q3 AON7524, Q4 AON7524, Q5 AON7423, U1 TSC213, U2 STC4054GR

Commit message: ACwing silkscreen: logos, board names, author, connector labels (DRC clean)
Co-Authored-By: Claude Opus 5.5 <noreply@anthropic.com>
Claude-Session: https://claude.ai/code/session_0189Xg6tRAL4bRZ656VQBtPX
Parts:
- added LOGO1: ACwing_Logo_Full_6mm, ACwing:ACwing_Logo_Full_6mm, F.Cu at (160.0, 84.2)
- added LOGO2: ACwing_Logo_Full_10mm, ACwing:ACwing_Logo_Full_10mm, B.Cu at (149.9, 97.3)
Other:
- board text added: "ACwing ESC 1S rev B"
- board text added: "Andrea Cirillo 2026"
- board text added: "CHARGE"
- board text added: "ESC 1S rev B"
- board text added: "TO FC"
- board text removed: "1S power board"
- board text removed: "ACwing ESC1S B"

Commit message: Reorganize docs, regenerate outputs, remove author name from the PCBs
- fabrication outputs, schematics, STEP and PCB views moved to 00 - Docs/<board>_Docs
- single mechanical handoff and stack check in 04 - System_Docs, brand files in 05 - Brand
- silkscreen: ACwing logo, board name and labels only (no author name)

Co-Authored-By: Claude Opus 5.5 <noreply@anthropic.com>
Claude-Session: https://claude.ai/code/session_0189Xg6tRAL4bRZ656VQBtPX
Parts:
- moved LOGO2 0.65 mm to (149.9, 98.0)
Other:
- board text removed: "Andrea Cirillo 2026"
