File: 02 - ESC_1S_KiCadProj/ACwing_ESC1S_B.kicad_sch (KiCad schematic)
At the start: 49 parts, among them J1 ESC link, J2 BATT 1S, J4 USB-C (HRO TYPE-C-31-M-12), M1 coreless 8520, M2 coreless 8520, M3 coreless 8520, M4 coreless 8520, Q1 AON7524, Q2 AON7524, Q3 AON7524, Q4 AON7524, Q5 AON7423, U1 TSC213, U2 STC4054GR

Commit message: Reorganize docs, regenerate outputs, remove author name from the PCBs
- fabrication outputs, schematics, STEP and PCB views moved to 00 - Docs/<board>_Docs
- single mechanical handoff and stack check in 04 - System_Docs, brand files in 05 - Brand
- silkscreen: ACwing logo, board name and labels only (no author name)

Co-Authored-By: Claude Opus 5.5 <noreply@anthropic.com>
Claude-Session: https://claude.ai/code/session_0189Xg6tRAL4bRZ656VQBtPX
Other:
- title: ACwing ESC1S rev B - ACwing 1S power board (brushed) for ACwing FC rev H -> ACwing ESC 1S rev B - 1S brushed power board with USB-C charger, for ACwing FC rev H
Changed lines of the file:
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@@
   (paper "A3")
   (title_block
-    (title "ACwing ESC1S rev B - ACwing 1S power board (brushed) for ACwing FC rev H")
-    (date "2026-10-18")
+    (title "ACwing ESC 1S rev B - 1S brushed power board with USB-C charger, for ACwing FC rev H")
+    (date "2026-10-19")
     (rev "B")
     (company "ACwing - Andrea Cirillo")
-    (comment 1 "40 x 40 mm, 2 layers, 1.0 mm; frame C outline; 20 x 20 mm M2 holes (hard mount)")
+    (comment 1 "40 x 40 mm, 4 layers, 1.0 mm; frame C outline; 20 x 20 mm M2 holes (hard mount)")
     (comment 2 "FC link: standard 4-in-1 ESC connector, JST SH 8-pin, 1:1 cable")
     (comment 3 "Larger drones: a commercial 4-in-1 ESC replaces this board on the same FC cable")
