File: 02 - ESC_1S_KiCadProj/ACwing_ESC1S_A.kicad_pcb (KiCad board)
At the start: 4 copper layers, 40.8 x 40.8 mm, 51 parts, among them J1 ESC link, J2 BATT 1S, J4 USB-C (HRO TYPE-C-31-M-12), M1 coreless 8520, M2 coreless 8520, M3 coreless 8520, M4 coreless 8520, Q1 AON7524, Q2 AON7524, Q3 AON7524, Q4 AON7524, Q5 AON7423, U1 TSC213, U2 STC4054GR

Commit message: Silkscreen review: board names, connector labels on the right side
- Board name + revision only, same on every board and layer: "FC rev A",
  "ESC 1S rev A", "GPS rev A", "Flow rev A" (was "ACwing ... rev A" on some).
- FC: USB and ESC A labels moved to the top (with J1 / J2); GPS and FLOW
  centred on J3 / J4; ESC B and ELRS on one line; BAT beside J7 / J8.
- Same fix on ESC 1S (CHARGE to the top, TO FC centred on J1) and GPS
  (QWIIC IN / OUT to the top, outside the SAM-M10Q outline).
- silk_brand.py: labels stay on the connector's side and never under a part;
  brand README rules updated. Gerbers, DRC (0 / 0 on all boards), views.

Co-Authored-By: Claude Opus 5.5 <noreply@anthropic.com>
Claude-Session: https://claude.ai/code/session_0189Xg6tRAL4bRZ656VQBtPX
Other:
- board text removed: "ACwing ESC 1S rev A"
Changed lines of the file:
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@@
   (gr_line (start 129.199999 87.7) (end 130 88.5)
     (stroke (width 0.1) (type default)) (layer "Edge.Cuts"))
-  (gr_text "CHARGE" (at 134.233 84.233) (layer "B.SilkS")
-    (effects (font (size 0.8 0.8) (thickness 0.15)) (justify mirror))
-  )
-  (gr_text "ACwing ESC 1S rev A" (at 149.883095 103.75) (layer "B.SilkS")
+  (gr_text "ESC 1S rev A" (at 149.883 103.75) (layer "B.SilkS")
     (effects (font (size 0.8 0.8) (thickness 0.15)) (justify mirror))
   )
@@
   (gr_text "+" (at 167.786969 103.009538) (layer "F.SilkS")
     (effects (font (size 0.9 0.9) (thickness 0.15)))
+  )
+  (gr_text "CHARGE" (at 138.65 88.247372 45) (layer "F.SilkS")
+    (effects (font (size 0.8 0.8) (thickness 0.15)))
   )
   (gr_text "M4 CW" (at 150 94.6) (layer "F.SilkS")
@@
     (effects (font (size 0.9 0.9) (thickness 0.15)))
   )
-  (gr_text "TO FC" (at 155.903971 112.470244) (layer "F.SilkS")
+  (gr_text "TO FC" (at 159.6 112.5) (layer "F.SilkS")
     (effects (font (size 0.8 0.8) (thickness 0.15)))
   )
