File: 02 - ESC_1S_KiCadProj/ACwing_ESC1S_A.kicad_pcb (KiCad board)
At the start: 4 copper layers, 40.8 x 40.8 mm, 51 parts, among them J1 ESC link, J2 BATT 1S, J4 USB-C (HRO TYPE-C-31-M-12), M1 coreless 8520, M2 coreless 8520, M3 coreless 8520, M4 coreless 8520, Q1 AON7524, Q2 AON7524, Q3 AON7524, Q4 AON7524, Q5 AON7423, U1 TSC213, U2 STC4054GR

Commit message: Removed references of the passive components and of the ICs on the top and bottom silkscreen. Left only the labels of the connectors.
Parts:
- moved LOGO1 4.65 mm to (164.6, 84.9)
- moved LOGO2 1.40 mm to (149.9, 99.4)
Other:
- board text added: "M1"
