File: 03 - GPS_KiCadProj/ACwing_GPS_D.kicad_pcb (KiCad board)
At the start: 2 copper layers, 30 x 30 mm, 26 parts, among them J1 Qwiic IN, J2 Qwiic OUT, Q1 2N7002, U1 SAM-M10Q-00B, U3 IIS2MDC

Commit message: ACwing silkscreen: logos, board names, author, connector labels (DRC clean)
Co-Authored-By: Claude Opus 5.5 <noreply@anthropic.com>
Claude-Session: https://claude.ai/code/session_0189Xg6tRAL4bRZ656VQBtPX
Parts:
- added LOGO1: ACwing_Logo_Full_5mm, ACwing_GPS:ACwing_Logo_Full_5mm, F.Cu at (138.7, 99.9)
- added LOGO2: ACwing_Logo_Full_7mm, ACwing_GPS:ACwing_Logo_Full_7mm, B.Cu at (146.1, 91.2)
Other:
- board text added: "ACwing GPS rev D"
- board text added: "GPS rev D"
- board text added: "QWIIC IN"
- board text added: "QWIIC OUT"
- board text removed: "ACwing GPS D"
