File: 03 - GPS_KiCadProj/ACwing_GPS_D.kicad_sch (KiCad schematic)
At the start: 26 parts, among them J1 Qwiic IN, J2 Qwiic OUT, Q1 2N7002, U1 SAM-M10Q-00B, U3 IIS2MDC

Commit message: Reorganize docs, regenerate outputs, remove author name from the PCBs
- fabrication outputs, schematics, STEP and PCB views moved to 00 - Docs/<board>_Docs
- single mechanical handoff and stack check in 04 - System_Docs, brand files in 05 - Brand
- silkscreen: ACwing logo, board name and labels only (no author name)

Co-Authored-By: Claude Opus 5.5 <noreply@anthropic.com>
Claude-Session: https://claude.ai/code/session_0189Xg6tRAL4bRZ656VQBtPX
Other:
- title: ACwing GPS rev D - GNSS + compass for ACwing FC H -> ACwing GPS rev D - GNSS + compass expansion for ACwing FC rev H
Changed lines of the file:
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@@
   (paper "A4")
   (title_block
-    (title "ACwing GPS rev D - GNSS + compass for ACwing FC H")
+    (title "ACwing GPS rev D - GNSS + compass expansion for ACwing FC rev H")
     (date "2026-10-19")
     (rev "D")
     (company "ACwing - Andrea Cirillo")
-    (comment 1 "30 x 30 mm, 2 layers, 1.0 mm; same 20 x 20 hole pattern as the flight controller rev F")
-    (comment 2 "Expansion bus: Qwiic (JST SH 4-pin) x 2, pass-through, from FC J3; daisy-chain to the flow board")
+    (comment 1 "30 x 30 mm, 2 layers, 1.0 mm; same 20 x 20 mm hole pattern as the flight controller")
+    (comment 2 "Expansion bus: Qwiic (JST SH 4-pin) x 2, pass-through, from FC J3; optional daisy-chain to the flow board")
     (comment 3 "u-blox SAM-M10Q (integrated patch antenna, pin compatible with SAM-M8Q)")
     (comment 4 "Generated automatically: run ERC before release"))
