File: 03 - GPS_KiCadProj/ACwing_GPS_A.kicad_sch (KiCad schematic)
At the start: 26 parts, among them J1 Qwiic IN, J2 Qwiic OUT, Q1 2N7002, U1 SAM-M10Q-00B, U3 IIS2MDC

Commit message: FC/GPS layout update (still rev A): MCU centred, J6 on the front edge, buck on the left edge, EMI fixes
- FC: MCU at the board centre, IMU south of it (rot 270, axes remapped in firmware), ESC link B J6 next to J5 on
  the front edge, input buck L3/U12 on the left edge (out of the corner between the rear LEDs)
- FC: LEDs D3/D4 rotated, LED supply pre-routed away from the magnetometer; EMI check script and results
- GPS: Qwiic J1 moved to v = +3.6, right above FC J3
- re-routed, DRC 0 on both boards; Gerber, STEP, PDF, BoM/CPL, views, stack check regenerated; docs updated

Co-Authored-By: Claude Opus 5.5 <noreply@anthropic.com>
Claude-Session: https://claude.ai/code/session_0189Xg6tRAL4bRZ656VQBtPX
Parts:
- J1: Note JST SH 1.0 mm 4-pin side entry, TOP side (rev A), right edg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 -> JST SH 1.0 mm 4-pin side entry, TOP side, right edge at v =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
- J2: Note JST SH 1.0 mm 4-pin side entry, TOP side (rev A), rear edge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 -> JST SH 1.0 mm 4-pin side entry, TOP side, rear edge (mouth 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
Changed lines of the file:
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@@
   (title_block
     (title "ACwing GPS rev A - GNSS + compass expansion for ACwing FC rev A")
-    (date "2026-10-19")
+    (date "2026-10-24")
     (rev "A")
     (company "ACwing - Andrea Cirillo")
@@
         (font
           (size 1.27 1.27)) hide))
-    (property "Note" "JST SH 1.0 mm 4-pin side entry, TOP side (rev A), right edge (mouth toward +X). From FC J3"
+    (property "Note" "JST SH 1.0 mm 4-pin side entry, TOP side, right edge at v = +3.6 (aligned with FC J3), mouth toward +X. From FC J3"
       (at 35.56 38.1 0)
       (effects
@@
         (font
           (size 1.27 1.27)) hide))
-    (property "Note" "JST SH 1.0 mm 4-pin side entry, TOP side (rev A), rear edge (mouth toward -Y). Optional pass-through (the flow board has its own FC port J4)"
+    (property "Note" "JST SH 1.0 mm 4-pin side entry, TOP side, rear edge (mouth toward -Y). Optional pass-through (the flow board has its own FC port J4)"
       (at 68.58 38.1 0)
       (effects
