File: 03 - GPS_KiCadProj/ACwing_GPS_A.kicad_pcb (KiCad board)
At the start: 2 copper layers, 30 x 30 mm, 28 parts, among them J1 Qwiic IN, J2 Qwiic OUT, Q1 2N7002, U1 SAM-M10Q-00B, U3 IIS2MDC

Commit message: FC/GPS layout update (still rev A): MCU centred, J6 on the front edge, buck on the left edge, EMI fixes
- FC: MCU at the board centre, IMU south of it (rot 270, axes remapped in firmware), ESC link B J6 next to J5 on
  the front edge, input buck L3/U12 on the left edge (out of the corner between the rear LEDs)
- FC: LEDs D3/D4 rotated, LED supply pre-routed away from the magnetometer; EMI check script and results
- GPS: Qwiic J1 moved to v = +3.6, right above FC J3
- re-routed, DRC 0 on both boards; Gerber, STEP, PDF, BoM/CPL, views, stack check regenerated; docs updated

Co-Authored-By: Claude Opus 5.5 <noreply@anthropic.com>
Claude-Session: https://claude.ai/code/session_0189Xg6tRAL4bRZ656VQBtPX
Parts:
- LOGO2: value ACwing_Logo_Full_7mm -> ACwing_Logo_Full_6mm; footprint ACwing_GPS:ACwing_Logo_Full_7mm -> ACwing_GPS:ACwing_Logo_Full_6mm
- moved LOGO2 19.0 mm to (147.2, 110.2)
- moved J1 3.60 mm to (161.9, 96.4)
Routing:
- net +3V3: track 64.6 -> 99.2 mm, vias 6 -> 3
- net I2C_SDA: track 49.4 -> 43.7 mm
- net PPS: track 13.5 -> 10.2 mm
- net I2C_SCL: track 43.5 -> 42.2 mm
- net GPS_RXD: track 34.0 -> 32.9 mm
- net SAFEBOOT_N: track 26.7 -> 27.6 mm
- net GND: track 10.8 -> 11.7 mm, vias 122 -> 113
- net RESET_N: track 16.1 -> 16.8 mm
- net GPS_TXD: track 35.4 -> 34.9 mm
Other:
- board text removed: "GPS rev A"

Commit message: Silkscreen review: board names, connector labels on the right side
- Board name + revision only, same on every board and layer: "FC rev A",
  "ESC 1S rev A", "GPS rev A", "Flow rev A" (was "ACwing ... rev A" on some).
- FC: USB and ESC A labels moved to the top (with J1 / J2); GPS and FLOW
  centred on J3 / J4; ESC B and ELRS on one line; BAT beside J7 / J8.
- Same fix on ESC 1S (CHARGE to the top, TO FC centred on J1) and GPS
  (QWIIC IN / OUT to the top, outside the SAM-M10Q outline).
- silk_brand.py: labels stay on the connector's side and never under a part;
  brand README rules updated. Gerbers, DRC (0 / 0 on all boards), views.

Co-Authored-By: Claude Opus 5.5 <noreply@anthropic.com>
Claude-Session: https://claude.ai/code/session_0189Xg6tRAL4bRZ656VQBtPX
Other:
- board text added: "GPS rev A"
- board text removed: "ACwing GPS rev A"
Changed lines of the file:
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@@
   (gr_arc (start 137 115) (mid 135.585786 114.414213) (end 135 113)
     (stroke (width 0.1) (type default)) (layer "Edge.Cuts"))
-  (gr_text "QWIIC OUT" (at 154.25 111.875) (layer "B.SilkS")
+  (gr_text "GPS rev A" (at 147.155 114) (layer "B.SilkS")
     (effects (font (size 0.8 0.8) (thickness 0.15)) (justify mirror))
   )
-  (gr_text "ACwing GPS rev A" (at 147.154523 114) (layer "B.SilkS")
-    (effects (font (size 0.8 0.8) (thickness 0.15)) (justify mirror))
+  (gr_text "QWIIC OUT" (at 142.823851 111.818826) (layer "F.SilkS")
+    (effects (font (size 0.8 0.8) (thickness 0.15)))
   )
-  (gr_text "QWIIC IN" (at 160.938093 101.311436) (layer "F.SilkS")
+  (gr_text "QWIIC IN" (at 161.7 91.74641) (layer "F.SilkS")
     (effects (font (size 0.8 0.8) (thickness 0.15)))
   )
@@
     (effects (font (size 0.8 0.8) (thickness 0.15)) (justify right))
   )
-  (gr_text "ACwing GPS rev A" (at 152.6 86.6) (layer "F.SilkS")
+  (gr_text "GPS rev A" (at 152.6 86.6) (layer "F.SilkS")
     (effects (font (size 0.8 0.8) (thickness 0.15)))
   )
