File: 04 - FLOW_KiCadProj/ACwing_Flow_A.kicad_sch (KiCad schematic)
At the start: 37 parts, among them J1 Qwiic, J2 Qwiic, U1 PMW3901MB-TXQT, U2 LDK130PU-R, U3 VL53L1CXV0FY/1, U4 STM32C011F4U6

Commit message: Reorganize docs, regenerate outputs, remove author name from the PCBs
- fabrication outputs, schematics, STEP and PCB views moved to 00 - Docs/<board>_Docs
- single mechanical handoff and stack check in 04 - System_Docs, brand files in 05 - Brand
- silkscreen: ACwing logo, board name and labels only (no author name)

Co-Authored-By: Claude Opus 5.5 <noreply@anthropic.com>
Claude-Session: https://claude.ai/code/session_0189Xg6tRAL4bRZ656VQBtPX
Other:
- title: ACwing Flow rev A - flow + ToF expansion -> ACwing Flow rev A - optical flow + ToF expansion for ACwing FC rev H
Changed lines of the file:
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@@
   (paper "A4")
   (title_block
-    (title "ACwing Flow rev A - flow + ToF expansion")
-    (date "2026-10-18")
+    (title "ACwing Flow rev A - optical flow + ToF expansion for ACwing FC rev H")
+    (date "2026-10-19")
     (rev "A")
     (company "ACwing - Andrea Cirillo")

Commit message: Release naming: all boards become rev A
- FC H, ESC 1S B, GPS D renamed to rev A (files, title blocks, silkscreen, BoM titles, docs); Flow stays rev A
- earlier pre-release iterations are called drafts in the docs (never manufactured)
- Gerber, STEP, schematic PDFs, DRC reports and PCB views regenerated (DRC 0 on all boards)

Co-Authored-By: Claude Opus 5.5 <noreply@anthropic.com>
Claude-Session: https://claude.ai/code/session_0189Xg6tRAL4bRZ656VQBtPX
Other:
- title: ACwing Flow rev A - optical flow + ToF expansion for ACwing FC rev H -> ACwing Flow rev A - optical flow + ToF expansion for ACwing FC rev A
Changed lines of the file:
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@@
   (paper "A4")
   (title_block
-    (title "ACwing Flow rev A - optical flow + ToF expansion for ACwing FC rev H")
+    (title "ACwing Flow rev A - optical flow + ToF expansion for ACwing FC rev A")
     (date "2026-10-19")
     (rev "A")
