File: 04 - FLOW_KiCadProj/ACwing_Flow_A.kicad_pcb (KiCad board)
At the start: 2 copper layers, 21 x 25 mm, 37 parts, among them J1 Qwiic, J2 Qwiic, U1 PMW3901MB-TXQT, U2 LDK130PU-R, U3 VL53L1CXV0FY/1, U4 STM32C011F4U6

Commit message: ACwing silkscreen: logos, board names, author, connector labels (DRC clean)
Co-Authored-By: Claude Opus 5.5 <noreply@anthropic.com>
Claude-Session: https://claude.ai/code/session_0189Xg6tRAL4bRZ656VQBtPX
Parts:
- added LOGO1: ACwing_Logo_Full_9mm, ACwing_Flow:ACwing_Logo_Full_9mm, B.Cu at (150.0, 97.3)
Other:
- board text added: "Andrea Cirillo 2026"
- board text removed: "UAV Control 2026"

Commit message: Reorganize docs, regenerate outputs, remove author name from the PCBs
- fabrication outputs, schematics, STEP and PCB views moved to 00 - Docs/<board>_Docs
- single mechanical handoff and stack check in 04 - System_Docs, brand files in 05 - Brand
- silkscreen: ACwing logo, board name and labels only (no author name)

Co-Authored-By: Claude Opus 5.5 <noreply@anthropic.com>
Claude-Session: https://claude.ai/code/session_0189Xg6tRAL4bRZ656VQBtPX
Parts:
- moved LOGO1 0.66 mm to (150.1, 98.0)
Other:
- board text removed: "Andrea Cirillo 2026"
Changed lines of the file:
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@@
   )
   (footprint "ACwing_Flow:ACwing_Logo_Full_9mm" locked (layer "B.Cu")
-    (at 149.956906 97.35 180)
-    (descr "ACwing full logo on the silkscreen, 9 mm high (Andrea Cirillo)")
+    (at 150.056905 98 180)
+    (descr "ACwing full logo on the silkscreen, 9 mm high")
     (tags "logo ACwing")
     (attr board_only exclude_from_pos_files exclude_from_bom)
@@
     (effects (font (size 0.8 0.8) (thickness 0.15)) (justify mirror))
   )
-  (gr_text "Andrea Cirillo 2026" (at 149.956906 103.75) (layer "B.SilkS")
+  (gr_text "ACwing Flow rev A" (at 150.056905 103.25) (layer "B.SilkS")
     (effects (font (size 0.8 0.8) (thickness 0.15)) (justify mirror))
   )
-  (gr_text "ACwing Flow rev A" (at 149.956906 102.6) (layer "B.SilkS")
-    (effects (font (size 0.8 0.8) (thickness 0.15)) (justify mirror))
-  )

Commit message: Silkscreen review: board names, connector labels on the right side
- Board name + revision only, same on every board and layer: "FC rev A",
  "ESC 1S rev A", "GPS rev A", "Flow rev A" (was "ACwing ... rev A" on some).
- FC: USB and ESC A labels moved to the top (with J1 / J2); GPS and FLOW
  centred on J3 / J4; ESC B and ELRS on one line; BAT beside J7 / J8.
- Same fix on ESC 1S (CHARGE to the top, TO FC centred on J1) and GPS
  (QWIIC IN / OUT to the top, outside the SAM-M10Q outline).
- silk_brand.py: labels stay on the connector's side and never under a part;
  brand README rules updated. Gerbers, DRC (0 / 0 on all boards), views.

Co-Authored-By: Claude Opus 5.5 <noreply@anthropic.com>
Claude-Session: https://claude.ai/code/session_0189Xg6tRAL4bRZ656VQBtPX
Other:
- board text added: "Flow rev A"
- board text removed: "ACwing Flow rev A"
Changed lines of the file:
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@@
     (effects (font (size 0.8 0.8) (thickness 0.15)) (justify mirror))
   )
-  (gr_text "ACwing Flow rev A" (at 150.056905 103.25) (layer "B.SilkS")
+  (gr_text "Flow rev A" (at 150.057 103.25) (layer "B.SilkS")
     (effects (font (size 0.8 0.8) (thickness 0.15)) (justify mirror))
   )
