File: 04 - FLOW_KiCadProj/ACwing_Flow_A.kicad_pcb (KiCad board)
At the start: 2 copper layers, 21 x 25 mm, 38 parts, among them J1 Qwiic, J2 Qwiic, U1 PMW3901MB-TXQT, U2 LDK130PU-R, U3 VL53L1CXV0FY/1, U4 STM32C011F4U6

Commit message: Removed references of the passive components and of the ICs on the top and bottom silkscreen. Left only the labels of the connectors.
Other:
- board text removed: "Qwiic J1 / J2"
